File: hardware/final_outline.kicad_pcb (KiCad board)
At the start: 2 copper layers, 99.5 x 75 mm, 36 parts, among them P1 CANCONNECTOR, P100 ISP, P101 DEBUG_LED, P2 CONN_01X14, U1 LM358N, U401 MCP2551-I/SN, U403 LPC11C14, U501 MCP1755-33, U502 MCP1755-5, U503 Zsr1000gta

Commit message: throttle interface pcb with additional TPS level converters
Parts:
- added C1: 1μ, Capacitors_SMD:C_0603_HandSoldering, F.Cu at (174.5, 103.1)
- added C2: 1μ, Capacitors_SMD:C_0603_HandSoldering, F.Cu at (177.3, 78.5)
- added G***: OSHW-logo_silkscreen-front_10mm, OSHW-logo:OSHW-logo_silkscreen-front_10mm, F.Cu at (196.1, 118.9)
- added G***: LOGO, MITEVT_LOGO:EVT-LOGO, F.Cu at (196.1, 106.4)
- added R6: 33k, Resistors_SMD:R_0603_HandSoldering, F.Cu at (185.7, 86.9)
- added R7: 47k, Resistors_SMD:R_0603_HandSoldering, F.Cu at (185.7, 84.3)
- added R8: 33k, Resistors_SMD:R_0603_HandSoldering, F.Cu at (171.4, 85.6)
- added R9: 47k, Resistors_SMD:R_0603_HandSoldering, F.Cu at (171.4, 88.4)
- added U2: LM358N, Housings_SOIC:SOIC-8_3.9x4.9mm_Pitch1.27mm, F.Cu at (178.3, 86.1)
- moved R2 5.64 mm to (166.1, 94.7)
- moved U1 5.54 mm to (173.0, 96.5)
- moved R4 5.41 mm to (179.8, 95.8)
- moved R5 5.34 mm to (179.8, 98.3)
- moved R3 4.89 mm to (166.1, 97.8)
- moved C505 3.86 mm to (159.4, 103.5)
- moved C506 3.81 mm to (155.6, 104.1)
- moved P1 2.50 mm to (123.2, 122.5)
- moved P2 2.44 mm to (165.0, 114.3)
- moved C502 0.48 mm to (135.1, 103.9)
- moved C501 0.27 mm to (135.1, 106.4)
Connections:
- P2 pad 10: Net-(P2-Pad10) -> +5V
- P2 pad 11: Net-(P2-Pad11) -> /BACK_PANEL/TPS4_5V
- P2 pad 12: Net-(P2-Pad12) -> GND
- P2 pad 7: Net-(P2-Pad7) -> +5V
- P2 pad 8: Net-(P2-Pad8) -> /BACK_PANEL/TPS3_5V
- P2 pad 9: Net-(P2-Pad9) -> GND
- U403 pad 34: /Micro_Controller/PIO1_1 -> /Micro_Controller/TPS3_3.3V
- U403 pad 35: /Micro_Controller/PIO1_2 -> /Micro_Controller/TPS4_3.3V
Routing:
- net (no net): track 0.75 -> 373.7 mm, vias 1 -> 0
- net /Micro_Controller/TPS3_3.3V: track 0.00 -> 69.4 mm, vias 0 -> 4
- net /Micro_Controller/TPS2_3.3V: track 2.64 -> 63.0 mm, vias 0 -> 4
- net /BACK_PANEL/TPS4_5V: track 0.00 -> 52.5 mm, vias 0 -> 2
- net /Micro_Controller/TPS4_3.3V: track 0.00 -> 49.0 mm, vias 0 -> 2
- net /BACK_PANEL/TPS3_5V: track 0.00 -> 44.9 mm, vias 0 -> 2
- net /Micro_Controller/TPS1_3.3V: track 3.84 -> 48.3 mm, vias 0 -> 2
- net GND: track 29.1 -> 50.2 mm, vias 6 -> 14
- net +5V: track 165.5 -> 182.4 mm, vias 2 -> 3
- net /BACK_PANEL/TPS1_5V: track 26.7 -> 19.5 mm
- net Net-(R6-Pad1): track 0.00 -> 4.89 mm
- net /BACK_PANEL/TPS2_5V: track 22.8 -> 18.1 mm
- net +12V: track 42.1 -> 46.5 mm
- net Net-(R8-Pad1): track 0.00 -> 4.38 mm
- net /FRONT_PANEL/LED6: track 22.9 -> 20.1 mm
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Other:
- board text added: "Throttle Interface"
